File: Echo_locator_Sensor_systems/Echo locator.brd (EAGLE design)
At the start: 62.2 x 49.2 mm, 48 parts, among them Q1 MOSFET-NCHANNEL2N7002PW, U1 MAX202CSE+

Commit message: Updated Board design Files
Parts:
- removed 10NF: 10nf, rcl:C0805
- added C1, C3: (no value), rcl:C0805
- C10, C4: value 1.2uf -> (none)
- C11, C12: value 22pf -> (none)
- C13, C14, C15, C18, C8: value 100nf -> (none)
- C16, C6: value 10nf -> (none)
- C2: value 1nf -> (none)
- C5: value 1n -> (none)
- C7: value 12pf -> (none)
- R1: value 62k -> (none)
- R10: value 75k -> (none)
- R11, R12, R18, R19, R22, R6, R7: value 10k -> (none)
- R13, R14, R16, R17: value 1k -> (none)
- R15: value 75 -> (none)
- R2: value 2.2k -> (none)
- R23: value 18k -> (none)
- R24, R4: value 120k -> (none)
- R5: value 3.3m -> (none)
- R8: value 3.9k -> (none)
- R9: value 4.53k -> (none)
- moved C18 15.3 mm to (52.7, 29.8), turned to 180 degrees
- moved C5 6.35 mm to (3.81, 5.71)
- moved R3 5.75 mm to (15.9, 14.0)
- moved R16 5.08 mm to (25.4, 4.45)
- moved C2 4.62 mm to (12.1, 4.45)
- moved C7 4.02 mm to (11.4, 8.26)
- moved R17 3.17 mm to (26.7, 13.3)
- moved R2 2.54 mm to (3.81, 13.3)
- moved R23 2.54 mm to (12.7, 13.3)
- moved R1 2.29 mm to (6.35, 10.8)
- moved R6 2.29 mm to (15.2, 10.8)
- moved C4 1.91 mm to (29.2, 8.89), turned to 270 degrees
- moved C14 1.27 mm to (46.4, 21.6)
- moved C15 0.64 mm to (51.4, 14.6), turned to 0 degrees
Connections:
- net N$15 renamed PA2
- net N$24 renamed PA3
- net N$25 renamed PA0
- net N$27 renamed PB0
- net N$29 renamed ICP
- net N$3 renamed PA1
- net N$31 renamed PB1
- net N$41 renamed C1+
- removed net +5V: OP-AMP.4
- removed net PE: C15.2, C18.1, PNP.C, U1.15, U1.16
- removed net VS+: C4.1
- new net WIRE: C1.2, C18.1, PNP.C, U1.16
- net GND: now also C1.1, C15.2, U1.15
- net N$1: now also C3.1; no longer 10NF.1
- net N$2: now also C3.2; no longer 10NF.2
- net VCC: now also C4.1, OP-AMP.4
Routing:
- net VCC: track 80.0 -> 177.7 mm, vias 6 -> 7
- net PE: track 42.1 -> 0.00 mm
- net GND: track 162.8 -> 194.5 mm, vias 4 -> 6
- net WIRE: track 0.00 -> 23.8 mm
- net PA1: track 98.7 -> 114.8 mm
- net N$12: track 18.7 -> 33.5 mm
- net PB1: track 39.6 -> 51.8 mm
- net PB0: track 37.0 -> 44.1 mm
- net N$49: track 13.0 -> 19.5 mm, vias 0 -> 1
- net N$46: track 12.1 -> 6.03 mm
- net N$21: track 4.14 -> 8.25 mm
- net N$8: track 13.7 -> 16.6 mm
- net N$3: track 6.93 -> 9.47 mm
- net N$7: track 2.36 -> 4.15 mm
- net N$44: track 3.01 -> 4.28 mm
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