File: Echo_locator_Sensor_systems/Echo locator.sch (EAGLE design)
At the start: 48 parts, among them Q1 MOSFET-NCHANNEL2N7002PW, U1 MAX202CSE+

Commit message: Updated Board design Files
Parts:
- added C1: (no value), rcl:C-USC0805
- C10, C4: value 1.2uf -> (none)
- C11, C12: value 22pf -> (none)
- C13, C14, C15, C18, C8: value 100nf -> (none)
- C16, C3, C6: value 10nf -> (none)
- C2: value 1nf -> (none)
- C5: value 1n -> (none)
- C7: value 12pf -> (none)
- R1: value 62k -> (none)
- R10: value 75k -> (none)
- R11, R12, R18, R19, R22, R6, R7: value 10k -> (none)
- R13, R14, R16, R17: value 1k -> (none)
- R15: value 75 -> (none)
- R2: value 2.2k -> (none)
- R23: value 18k -> (none)
- R24, R4: value 120k -> (none)
- R5: value 3.3m -> (none)
- R8: value 3.9k -> (none)
- R9: value 4.53k -> (none)
- renumbered 10NF to C3
Connections:
- net N$15 renamed PA2
- net N$24 renamed PA3
- net N$25 renamed PA0
- net N$27 renamed PB0
- net N$29 renamed ICP
- net N$3 renamed PA1
- net N$31 renamed PB1
- net N$41 renamed C1+
- removed net +5V: OP-AMP1.V+
- removed net PE: C15.2, C18.1, PNP.C, U1.GND, U1.VCC
- removed net VS+: C4.1
- new net WIRE: C1.2, C18.1, PNP.C, U1.VCC
- net GND: now also C1.1, C15.2, U1.GND
- net VCC: now also C4.1, OP-AMP1.V+
